File: eagle/pxbee-trigger.sch (EAGLE design)
At the start: 21 parts, among them J1 39501-1002, J2 39501-1009, K1 APAN3103, K2 APAN3103, K3 APAN3103, K4 APAN3103, Q1 BC548BTA, Q2 BC548BTA, Q3 BC548BTA, Q4 BC548BTA

Commit message: Added capacitors for fixing #12
- Version of the PCB updated to v0.3.0
Parts:
- added C1: EEU-FM1H221-A, parts:EEU-FM1H221-A
- added C2: EEU-FM1H221-A2, parts:EEU-FM1H221-A2
Connections:
- removed net N$10: BR1.-, PS1.-VIN
- removed net N$11: BR1.+, PS1.+VIN
- new net VIN+: BR1.+, C1.+, C2.+, PS1.+VIN
- new net VIN-: BR1.-, C1.-, C2.-, PS1.-VIN
Changed lines of the file:
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@@
 <?xml version="1.0" encoding="utf-8"?>
 <!DOCTYPE eagle SYSTEM "eagle.dtd">
-<eagle version="9.6.0">
+<eagle version="9.6.2">
 <drawing>
 <settings>
@@
 <grid distance="0.1" unitdist="inch" unit="inch" style="lines" multiple="1" display="no" altdistance="0.01" altunitdist="inch" altunit="inch"/>
 <layers>
-<layer number="1" name="Top" color="4" fill="1" visible="no" active="no"/>
-<layer number="16" name="Bottom" color="1" fill="1" visible="no" active="no"/>
-<layer number="17" name="Pads" color="2" fill="1" visible="no" active="no"/>
-<layer number="18" name="Vias" color="2" fill="1" visible="no" active="no"/>
-<layer number="19" name="Unrouted" color="6" fill="1" visible="no" active="no"/>
-<layer number="20" name="Dimension" color="15" fill="1" visible="no" active="no"/>
-<layer number="21" name="tPlace" color="7" fill="1" visible="no" active="no"/>
-<layer number="22" name="bPlace" color="7" fill="1" visible="no" active="no"/>
-<layer number="23" name="tOrigins" color="15" fill="1" visible="no" active="no"/>
-<layer number="24" name="bOrigins" color="15" fill="1" visible="no" active="no"/>
-<layer number="25" name="tNames" color="7" fill="1" visible="no" active="no"/>
-<layer number="26" name="bNames" color="7" fill="1" visible="no" active="no"/>
-<layer number="27" name="tValues" color="7" fill="1" visible="no" active="no"/>
-<layer number="28" name="bValues" color="7" fill="1" visible="no" active="no"/>
+<layer number="1" name="Top" color="4" fill="1" visible="yes" active="no"/>
+<layer number="16" name="Bottom" color="1" fill="1" visible="yes" active="no"/>
+<layer number="17" name="Pads" color="2" fill="1" visible="yes" active="no"/>
+<layer number="18" name="Vias" color="2" fill="1" visible="yes" active="no"/>
+<layer number="19" name="Unrouted" color="6" fill="1" visible="yes" active="no"/>
+<layer number="20" name="Dimension" color="24" fill="1" visible="yes" active="no"/>
+<layer number="21" name="tPlace" color="7" fill="1" visible="yes" active="no"/>
+<layer number="22" name="bPlace" color="7" fill="1" visible="yes" active="no"/>
+<layer number="23" name="tOrigins" color="15" fill="1" visible="yes" active="no"/>
+<layer number="24" name="bOrigins" color="15" fill="1" visible="yes" active="no"/>
+<layer number="25" name="tNames" color="7" fill="1" visible="yes" active="no"/>
+<layer number="26" name="bNames" color="7" fill="1" visible="yes" active="no"/>
+<layer number="27" name="tValues" color="7" fill="1" visible="yes" active="no"/>
+<layer number="28" name="bValues" color="7" fill="1" visible="yes" active="no"/>
 <layer number="29" name="tStop" color="7" fill="3" visible="no" active="no"/>
 <layer number="30" name="bStop" color="7" fill="6" visible="no" active="no"/>
@@
 <layer number="35" name="tGlue" color="7" fill="4" visible="no" active="no"/>
 <layer number="36" name="bGlue" color="7" fill="5" visible="no" active="no"/>
-<layer number="37" name="tTest" color="7" fill="1" visible="no" active="no"/>
-<layer number="38" name="bTest" color="7" fill="1" visible="no" active="no"/>
+<layer number="37" name="tTest" color="7" fill="1" visible="yes" active="no"/>
+<layer number="38" name="bTest" color="7" fill="1" visible="yes" active="no"/>
 <layer number="39" name="tKeepout" color="4" fill="11" visible="no" active="no"/>
 <layer number="40" name="bKeepout" color="1" fill="11" visible="no" active="no"/>
@@
 <layer number="44" name="Drills" color="7" fill="1" visible="no" active="no"/>
 <layer number="45" name="Holes" color="7" fill="1" visible="no" active="no"/>
-<layer number="46" name="Milling" color="3" fill="1" visible="no" active="no"/>
-<layer number="47" name="Measures" color="7" fill="1" visible="no" active="no"/>
-<layer number="48" name="Document" color="7" fill="1" visible="no" active="no"/>
-<layer number="49" name="Reference" color="7" fill="1" visible="no" active="no"/>
-<layer number="51" name="tDocu" color="7" fill="1" visible="no" active="no"/>
-<layer number="52" name="bDocu" color="7" fill="1" visible="no" active="no"/>
+<layer number="46" name="Milling" color="3" fill="1" visible="yes" active="no"/>
+<layer number="47" name="Measures" color="7" fill="1" visible="yes" active="no"/>
+<layer number="48" name="Document" color="7" fill="1" visible="yes" active="no"/>
+<layer number="49" name="Reference" color="7" fill="1" visible="yes" active="no"/>
+<layer number="51" name="tDocu" color="7" fill="1" visible="yes" active="no"/>
+<layer number="52" name="bDocu" color="7" fill="1" visible="yes" active="no"/>
 <layer number="88" name="SimResults" color="9" fill="1" visible="yes" active="yes"/>
 <layer number="89" name="SimProbes" color="9" fill="1" visible="yes" active="yes"/>
@@
 <part name="J1" library="parts" deviceset="39501-1002" device=""/>
 <part name="J2" library="parts" deviceset="39501-1009" device=""/>
+<part name="C1" library="parts" deviceset="EEU-FM1H221" device="-A" value="EEU-FM1H221-A"/>
+<part name="C2" library="parts" deviceset="EEU-FM1H221" device="-A2" value="EEU-FM1H221-A2"/>
 </parts>
 <sheets>
@@
 <attribute name="VALUE" x="45.72" y="29.21" size="1.778" layer="96" rot="R270" align="center-left"/>
 </instance>
+<instance part="C1" gate="G$1" x="7.62" y="104.14" smashed="yes">
+<attribute name="NAME" x="16.51" y="110.49" size="1.778" layer="95" align="center-left"/>
+<attribute name="VALUE" x="16.51" y="107.95" size="1.778" layer="96" align="center-left"/>
+</instance>
+<instance part="C2" gate="G$1" x="7.62" y="111.76" smashed="yes">
+<attribute name="NAME" x="16.51" y="118.11" size="1.778" layer="95" align="center-left"/>
+<attribute name="VALUE" x="16.51" y="115.57" size="1.778" layer="96" align="center-left"/>
+</instance>
 </instances>
 <busses>
@@
 </segment>
 </net>
-<net name="N$10" class="0">
+<net name="VIN-" class="0">
 <segment>
 <pinref part="BR1" gate="G$1" pin="-"/>
@@
 <wire x1="12.7" y1="73.66" x2="12.7" y2="99.06" width="0.1524" layer="91"/>
 <wire x1="12.7" y1="99.06" x2="20.32" y2="99.06" width="0.1524" layer="91"/>
-</segment>
-</net>
-<net name="N$11" class="0">
+<pinref part="C1" gate="G$1" pin="-"/>
+<wire x1="20.32" y1="104.14" x2="20.32" y2="99.06" width="0.1524" layer="91"/>
+<junction x="20.32" y="99.06"/>
+<pinref part="C2" gate="G$1" pin="-"/>
+<wire x1="20.32" y1="111.76" x2="20.32" y2="104.14" width="0.1524" layer="91"/>
+<junction x="20.32" y="104.14"/>
+</segment>
+</net>
+<net name="VIN+" class="0">
 <segment>
 <pinref part="BR1" gate="G$1" pin="+"/>
@@
 <wire x1="15.24" y1="73.66" x2="15.24" y2="96.52" width="0.1524" layer="91"/>
 <wire x1="15.24" y1="96.52" x2="20.32" y2="96.52" width="0.1524" layer="91"/>
-</segment>
-</net>
+<pinref part="C1" gate="G$1" pin="+"/>
+<wire x1="7.62" y1="104.14" x2="7.62" y2="96.52" width="0.1524" layer="91"/>
+<wire x1="7.62" y1="96.52" x2="15.24" y2="96.52" width="0.1524" layer="91"/>
+<junction x="15.24" y="96.52"/>
+<pinref part="C2" gate="G$1" pin="+"/>
+<wire x1="7.62" y1="111.76" x2="7.62" y2="104.14" width="0.1524" layer="91"/>
+<junction x="7.62" y="104.14"/>
+</segment>
+</net>

Commit message: UART header added for easier debugging
- Fixes #13
Parts:
- added JP1: (no value), SparkFun-Connectors:6_PIN_SERIAL_TARGETSILK
Connections:
- new net CTS: JP1.CTS, XB1.!CTS!/DIO7
- new net DTR: JP1.DTR, XB1.!DTR!/SLEEP_RQ/DIO8
- new net RXI: JP1.RXI, XB1.DIN/!CONFIG
- new net TXO: JP1.TXO, XB1.DOUT
- net GND: now also JP1.GND
- net VCC: now also JP1.VCC

Commit message: Bridge rectifier upgrade; XBee reset header
- [Parts] Bridge rectifier upgraded from DF005 to DF01, previous part was underdimensioned
- [SCH,BRD] Added J3 pinout for XBee Reset
- [BRD] Version bumped to v0.4.0
Parts:
- added J3: (no value), SparkFun-Connectors:CONN_02
- BR1: value DF005M -> DF01M; device parts:DF005M -> parts:DF01M
Connections:
- net DIO1 renamed STAT1
- net DIO2 renamed STAT2
- new net RST: J3.1, XB1.!RESET
- net GND: now also J3.2
Changed lines of the file:
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@@
 <parts>
 <part name="FRAME1" library="frames" library_urn="urn:adsk.eagle:library:229" deviceset="A4L-LOC" device=""/>
-<part name="BR1" library="parts" deviceset="DF005M" device=""/>
+<part name="BR1" library="parts" deviceset="DF01M" device=""/>
 <part name="PS1" library="parts" deviceset="MGFS1R5243R3" device=""/>
 <part name="XB1" library="xbee" deviceset="XBEE" device="-PRO"/>
@@
 <part name="C2" library="parts" deviceset="EEU-FM1H221" device="-A2" value="EEU-FM1H221-A2"/>
 <part name="JP1" library="SparkFun-Connectors" library_urn="urn:adsk.eagle:library:513" deviceset="6_PIN_SERIAL_TARGET" device="SILK" package3d_urn="urn:adsk.eagle:package:37995/1"/>
+<part name="J3" library="SparkFun-Connectors" library_urn="urn:adsk.eagle:library:513" deviceset="CONN_02" device="" package3d_urn="urn:adsk.eagle:package:38039/1"/>
 </parts>
 <sheets>
@@
 <attribute name="VALUE" x="80.01" y="7.62" size="1.778" layer="96"/>
 </instance>
+<instance part="J3" gate="G$1" x="109.22" y="22.86" smashed="yes">
+<attribute name="VALUE" x="106.68" y="18.034" size="1.778" layer="96" font="vector"/>
+<attribute name="NAME" x="106.68" y="28.448" size="1.778" layer="95" font="vector"/>
+</instance>
 </instances>
 <busses>
@@
 <wire x1="91.44" y1="25.4" x2="99.06" y2="25.4" width="0.1524" layer="91"/>
 <label x="93.726" y="25.654" size="1.778" layer="95"/>
+</segment>
+<segment>
+<pinref part="J3" gate="G$1" pin="2"/>
+<wire x1="116.84" y1="25.4" x2="127" y2="25.4" width="0.1524" layer="91"/>
+<label x="121.412" y="25.654" size="1.778" layer="95"/>
 </segment>
 </net>
@@
 </segment>
 </net>
-<net name="DIO2" class="0">
+<net name="STAT2" class="0">
 <segment>
 <pinref part="XB1" gate="G$1" pin="AD2/DIO2"/>
 <wire x1="55.88" y1="139.7" x2="55.88" y2="129.54" width="0.1524" layer="91"/>
-<label x="50.8" y="127" size="1.778" layer="95"/>
+<label x="48.26" y="127" size="1.778" layer="95"/>
 </segment>
 <segment>
@@
 </segment>
 </net>
-<net name="DIO1" class="0">
+<net name="STAT1" class="0">
 <segment>
 <pinref part="XB1" gate="G$1" pin="AD1/DIO1"/>
@@
 </segment>
 </net>
+<net name="RST" class="0">
+<segment>
+<pinref part="XB1" gate="G$1" pin="!RESET"/>
+<wire x1="22.86" y1="139.7" x2="22.86" y2="132.08" width="0.1524" layer="91"/>
+<label x="20.574" y="129.54" size="1.778" layer="95"/>
+</segment>
+<segment>
+<pinref part="J3" gate="G$1" pin="1"/>
+<wire x1="116.84" y1="22.86" x2="127" y2="22.86" width="0.1524" layer="91"/>
+<label x="121.666" y="23.114" size="1.778" layer="95"/>
+</segment>
+</net>
